Commit message: added joint to allow urdf of whole body to be shown correctly

File: urdf/ximu3.urdf.xacro (robot description, xacro)
@@ -40,3 +40,14 @@
 		</link>
 	</xacro:macro>
+	<xacro:macro name="ximu_joint" params="ximu3_name parent">
+		<joint name="${ximu3_name}_joint" type="fixed">
+			<origin xyz="0 0 1" rpy="0 0 0"/>
+			<parent link="${parent}"/>
+			<child link="${ximu3_name}"/>
+		</joint>
+	</xacro:macro>
+	<xacro:macro name="ximu_link_and_joint" params="parent">
+		<xacro:ximu_link ximu3_name="${parent}_imu"/>
+		<xacro:ximu_joint ximu3_name="${parent}_imu" parent="${parent}"/>
+	</xacro:macro>
 </robot>

Commit message: changed color, added params

File: urdf/ximu3.urdf.xacro (robot description, xacro)
@@ -26,5 +26,5 @@
 				</geometry>
 				<material name="">
-					<color	rgba="0.7921 0.8196 0.9333 1" />
+					<color	rgba="0.92 0.2 0.2 1" />
 				</material>
 			</visual>
@@ -40,14 +40,25 @@
 		</link>
 	</xacro:macro>
-	<xacro:macro name="ximu_joint" params="ximu3_name parent">
-		<joint name="${ximu3_name}_joint" type="fixed">
-			<origin xyz="0 0 1" rpy="0 0 0"/>
+	<xacro:macro name="ximu_joint_floating" params="ximu3_name parent origin">
+		<joint name="${ximu3_name}_joint" type="floating">
+			<origin xyz="${origin}" rpy="0 0 0"/>
 			<parent link="${parent}"/>
 			<child link="${ximu3_name}"/>
 		</joint>
 	</xacro:macro>
-	<xacro:macro name="ximu_link_and_joint" params="parent">
+	<xacro:macro name="ximu_joint" params="ximu3_name parent origin">
+		<joint name="${ximu3_name}_joint" type="fixed">
+			<origin xyz="${origin}" rpy="0 0 0"/>
+			<parent link="${parent}"/>
+			<child link="${ximu3_name}"/>
+		</joint>
+	</xacro:macro>
+	<xacro:macro name="ximu_link_and_joint" params="parent origin">
 		<xacro:ximu_link ximu3_name="${parent}_imu"/>
-		<xacro:ximu_joint ximu3_name="${parent}_imu" parent="${parent}"/>
+		<xacro:ximu_joint ximu3_name="${parent}_imu" parent="${parent}" origin="${origin}"/>
+	</xacro:macro>
+	<xacro:macro name="ximu_link_and_joint_floating" params="parent origin">
+		<xacro:ximu_link ximu3_name="${parent}_imu"/>
+		<xacro:ximu_joint_floating ximu3_name="${parent}_imu" parent="${parent}" origin="${origin}"/>
 	</xacro:macro>
 </robot>

Commit message: small visualization changes

File: urdf/ximu3.urdf.xacro (robot description, xacro)
@@ -1,5 +1,5 @@
-<?xml version="1.0" encoding="utf-8"?>
+<?xml version="0.0" encoding="utf-8"?>
 <robot xmlns:xacro="http://www.ros.org/wiki/xacro">
-	<xacro:macro name="ximu_link" params="ximu3_name">
+	<xacro:macro name="ximu_link" params="ximu3_name color:='0.92 0.2 0.2 1'">
 		<link name="${ximu3_name}" >
 			<inertial>
@@ -26,14 +26,13 @@
 				</geometry>
 				<material name="">
-					<color	rgba="0.92 0.2 0.2 1" />
+					<color	rgba="${color}" />
 				</material>
 			</visual>
 			<collision>
 				<origin
-					xyz="0 0 0"
+					xyz="0.003 0 -0.002"
 					rpy="0 0 0" />
 				<geometry>
-					<mesh
-						filename="package://ximu3_ros/meshes/housing_s.stl" />
+					<box size=".058 .05 .015" />
 				</geometry>
 			</collision>
@@ -57,8 +56,21 @@
 		<xacro:ximu_link ximu3_name="${parent}_imu"/>
 		<xacro:ximu_joint ximu3_name="${parent}_imu" parent="${parent}" origin="${origin}"/>
+		<xacro:ximu_sensor parent="${parent}"/>
 	</xacro:macro>
 	<xacro:macro name="ximu_link_and_joint_floating" params="parent origin">
 		<xacro:ximu_link ximu3_name="${parent}_imu"/>
 		<xacro:ximu_joint_floating ximu3_name="${parent}_imu" parent="${parent}" origin="${origin}"/>
+		<xacro:ximu_sensor parent="${parent}"/>
+	</xacro:macro>
+	<xacro:macro name="ximu_sensor" params="parent">
+		<sensor name="${parent}_sensor" update_rate="1" type="imu">
+			<origin xyz="0 0 0" rpy="0 0 0"/>
+			<imu>
+			</imu>
+		</sensor>
+	</xacro:macro>
+	<xacro:macro name="ximu_cal" params="parent origin">
+		<xacro:ximu_link ximu3_name="${parent}_0" color="0.2 0.2 0.2 1"/>
+		<xacro:ximu_joint ximu3_name="${parent}_0" parent="${parent}_base" origin="${origin}" />
 	</xacro:macro>
 </robot>
